File: pcb/little-chef.kicad_pcb (KiCad board)
At the start: 2 copper layers, 78 x 78 mm, 99 parts, among them J1 Conn_01x02, J2 Conn_01x06, J3 Conn_01x09, J4 USB_B_Mini, J5 Conn_01x06, J6 Conn_01x04, J7 Conn_01x07, J8 Conn_01x03, K1 G5LE-1, Q1 BSP75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

Commit message: Add first prototype
Parts:
- removed K1: G5LE-1, Relay_THT:Relay_SPDT_Omron-G5LE-1
- removed REF**: KiCad-Logo2_5mm_SilkScreen, Symbol:KiCad-Logo2_5mm_SilkScreen
- removed REF**: OSHW-Symbol_6.7x6mm_SilkScreen, Symbol:OSHW-Symbol_6.7x6mm_SilkScreen
- removed kibuzzard-63657C5D: G***, kibuzzard-63657C5D
- removed kibuzzard-63657C65: G***, kibuzzard-63657C65
- removed kibuzzard-63657C71: G***, kibuzzard-63657C71
- J8: value Conn_01x03 -> Conn_01x02; footprint Connector_PinHeader_2.54mm:PinHeader_1x03_P2.54mm_Vertical -> Connector_PinHeader_2.54mm:PinHeader_1x02_P2.54mm_Vertical
- moved D4 30.0 mm to (180.5, 121.5)
- moved Q4 26.9 mm to (172.0, 122.0)
- moved kibuzzard-63657DA3 1.28 mm to (190.0, 121.1)
- moved kibuzzard-63657DB8 0.27 mm to (190.0, 90.8)
Connections:
- D4 pad 2: Net-(D4-Pad2) -> /RELAY-
- J8 pad 1: Net-(J8-Pad1) -> VDC
- J8 pad 2: Net-(J8-Pad2) -> /RELAY-
- Q4 pad 2: Net-(D4-Pad2) -> /RELAY-
Routing:
- net Net-(D4-Pad2): track 43.4 -> 0.00 mm
- net Net-(J8-Pad3): track 33.2 -> 0.00 mm
- net Net-(J8-Pad1): track 29.7 -> 0.00 mm
- net /RELAY-: track 0.00 -> 18.9 mm
- net Net-(Q4-G): track 46.7 -> 62.8 mm, vias 2 -> 4
- net Net-(J8-Pad2): track 14.3 -> 0.00 mm
- net VDC: track 153.7 -> 166.6 mm
- net Net-(Q3-G): track 48.5 -> 45.3 mm
- net Net-(J3-Pin_8): track 47.3 -> 45.0 mm
Other:
- board text added: "Bottom Assembly View | Scale 1:1"
- board text added: "Top Assembly View | Scale 1:1"
- board text removed: "Bottom Assembly View | Scale 2:1"
- board text removed: "Top Assembly View | Scale 2:1"
