File: pcb/little-chef.kicad_sch (KiCad schematic)
At the start: 46 parts, among them J1 Conn_01x02, J2 Conn_01x06, J3 Conn_01x09, J4 USB_B_Mini, J5 Conn_01x06, J6 Conn_01x04, J7 Conn_01x07, J8 Conn_01x03, K1 G5LE-1, Q1 BSP75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

Commit message: Add first prototype
Parts:
- removed J8: Conn_01x03, Connector_PinHeader_2.54mm:PinHeader_1x03_P2.54mm_Vertical, symbol Connector_Generic:Conn_01x03
- removed K1: G5LE-1, Relay_THT:Relay_SPDT_Omron-G5LE-1, symbol Relay:G5LE-1
- added J8: Conn_01x02, Connector_PinHeader_2.54mm:PinHeader_1x02_P2.54mm_Vertical, symbol Connector_Generic:Conn_01x02
- H1, H2, H3, H4: now left out of the parts list
Connections:
- net VDC: now also J8.1 (Pin_1)
- net RELAY-: now reaches D4.2 (A), Q4.2 (D)
- net RELAY-: now also J8.2 (Pin_2)
Other:
- company: Made by CAZaugg -> Made by cazaugg
- moved on the sheet: D4
